Commit message: collisions fixed for panda hand

File: PandaStation/models/panda_hand_fixed_collisions.urdf (robot description, URDF)
Before this commit: robot hand, 3 links, 2 joints
Links:
- link panda_hand: geometry collision box size=0.062 0.20 0.066; collision box size=0.062 0.20 0.066
- link panda_leftfinger: geometry collision box size=0.017 0.014 0.017; collision box size=0.017 0.014 0.036
- link panda_rightfinger: geometry collision box size=0.017 0.014 0.017; collision box size=0.017 0.014 0.036
Joints:
- joint panda_finger_joint1: axis (none) -> 0 1 0; limit (none) -> lower=0.0 upper=0.04 effort=20 velocity=0.2; origin xyz=0 0.04 0.0584 rpy=0 0 0 -> xyz=0 0 0.0584 rpy=0 0 0; type fixed -> prismatic
- joint panda_finger_joint2: axis (none) -> 0 -1 0; limit (none) -> lower=0.0 upper=0.04 effort=20 velocity=0.2; mimic (none) -> joint=panda_finger_joint1; origin xyz=0 -0.04 0.0584 rpy=0 0 0 -> xyz=0 0 0.0584 rpy=0 0 0; type fixed -> prismatic

File: PandaStation/models/welded_panda_hand.urdf (robot description, URDF)
Before this commit: robot hand, 3 links, 2 joints
Links:
- link panda_hand: geometry collision box size=0.062 0.20 0.066; collision box size=0.062 0.20 0.066
- link panda_leftfinger: geometry collision box size=0.017 0.014 0.017; collision box size=0.017 0.014 0.036
- link panda_rightfinger: geometry collision box size=0.017 0.014 0.017; collision box size=0.017 0.014 0.036

Commit message: close to full stack

File: PandaStation/models/panda_hand_fixed_collisions.urdf (robot description, URDF)
Before this commit: robot hand, 3 links, 2 joints
Links:
- link panda_hand: geometry collision box size=0.062 0.20 0.066; collision box size=0.062 0.20 0.066
- link panda_leftfinger: geometry collision box size=0.017 0.014 0.017; collision box size=0.017 0.014 0.036
- link panda_rightfinger: geometry collision box size=0.017 0.014 0.017; collision box size=0.017 0.014 0.036

File: PandaStation/models/welded_panda_hand.urdf (robot description, URDF)
Before this commit: robot hand, 3 links, 2 joints
Links:
- link panda_hand: geometry collision box size=0.062 0.20 0.066; collision box size=0.062 0.20 0.066
- link panda_leftfinger: geometry collision box size=0.017 0.014 0.017; collision box size=0.017 0.014 0.036
- link panda_rightfinger: geometry collision box size=0.017 0.014 0.017; collision box size=0.017 0.014 0.036
