Commit message: sphere done

File: PandaStation/models/marble.urdf (robot description, URDF)
Before this commit: robot puck, 1 links, 0 joints
Links:
- link base_link: mass 1 -> 0.17; geometry collision sphere radius=0.03; visual sphere radius=0.03

File: PandaStation/models/puck.urdf (robot description, URDF)
Before this commit: robot puck, 1 links, 0 joints
Links:
- link base_link: mass 1 -> 0.17
