Commit message: omni hand

File: PandaStation/models/omni_arm.urdf (robot description, URDF)
Before this commit: robot omni_arm, 7 links, 6 joints
Joints:
- joint pitch_joint: limit lower=-3.14159265358979 upper=3.14159265358979 effort=87 velocity=3.141592 -> lower=-3.1416 upper=3.1416 effort=87 velocity=3.141592
- joint roll_joint: limit lower=-3.14159265358979 upper=3.14159265358979 effort=87 velocity=3.141592 -> lower=-3.1416 upper=3.1416 effort=87 velocity=3.141592
- joint yaw_joint: limit lower=-3.14159265358979 upper=3.14159265358979 effort=87 velocity=3.141592 -> lower=-3.1416 upper=3.1416 effort=87 velocity=3.141592

Commit message: improvments on floating hand

File: PandaStation/models/omni_arm.urdf (robot description, URDF)
Before this commit: robot omni_arm, 7 links, 6 joints
Joints:
- joint pitch_joint: limit lower=-3.1416 upper=3.1416 effort=87 velocity=3.141592 -> lower=0 upper=3.1416 effort=87 velocity=3.141592
- joint roll_joint: limit lower=-3.1416 upper=3.1416 effort=87 velocity=3.141592 -> lower=0 upper=3.1416 effort=87 velocity=3.141592
- joint yaw_joint: limit lower=-3.1416 upper=3.1416 effort=87 velocity=3.141592 -> lower=0 upper=3.1416 effort=87 velocity=3.141592
