Commit message: improved panda hand model and gripping constraints

File: PandaStation/models/puck.urdf (robot description, URDF)
Before this commit: robot puck, 1 links, 0 joints
Links:
- link base_link: mass 0.17 -> 0.1; geometry collision cylinder length=0.03 radius=0.03; visual cylinder length=0.03 radius=0.03
